File: ECI-Breakout.kicad_pcb (KiCad board)
At the start: 2 copper layers, 4 parts, among them P1 CONN_02X07

Commit message: First elaborate project
Parts:
- added OSHW: Symbol_OSHW-Logo_SilkScreen, Symbols:Symbol_OSHW-Logo_SilkScreen, B.Cu at (132.6, 97.0)
- added P2: CONN_01X07, Pin_Headers:Pin_Header_Straight_1x07, F.Cu at (139.7, 83.8)
- added kicadlogo: KiCad-Logo_5mm_SilkScreen, Symbol:KiCad-Logo_5mm_SilkScreen, B.Cu at (132.1, 91.9)
- P1: value CONN_02X07 -> CONN_01X07; footprint Connector_PinHeader_2.54mm:PinHeader_2x07_P2.54mm_Vertical -> Pin_Headers:Pin_Header_Straight_1x07
- R1: value 330 -> 1.5K; footprint Resistors_SMD:R_1210_HandSoldering -> Resistors_SMD:R_1206_HandSoldering
- moved P1 32.6 mm to (139.7, 73.7), turned to 270 degrees
- moved ECI1 29.6 mm to (122.4, 119.0)
- moved R1 21.9 mm to (127.0, 101.0)
- moved D1 14.1 mm to (135.0, 101.0), turned to 180 degrees
Connections:
- P1 pad 1: Net-(ECI1-Pad1) -> Net-(ECI1-PadA)
- P1 pad 2: GND -> Net-(ECI1-PadB)
- P1 pad 3: Net-(ECI1-Pad2) -> Net-(ECI1-PadC)
- P1 pad 4: Net-(ECI1-PadF) -> Net-(ECI1-PadD)
- P1 pad 5: Net-(ECI1-Pad3) -> Net-(ECI1-PadE)
- P1 pad 6: Net-(ECI1-PadE) -> Net-(ECI1-PadF)
- P1 pad 7: Net-(ECI1-Pad4) -> GND
Routing:
- net GND: track 0.00 -> 57.3 mm, vias 0 -> 2
- net Net-(ECI1-PadE): track 0.00 -> 52.5 mm
- net VCC: track 0.00 -> 50.9 mm
- net Net-(ECI1-PadD): track 0.00 -> 50.1 mm
- net Net-(ECI1-PadC): track 0.00 -> 48.0 mm
- net Net-(ECI1-PadB): track 0.00 -> 46.5 mm
- net Net-(ECI1-PadA): track 0.00 -> 45.7 mm
- net Net-(ECI1-PadF): track 0.00 -> 44.7 mm
- net Net-(ECI1-Pad6): track 0.00 -> 31.9 mm
- net Net-(ECI1-Pad1): track 0.00 -> 31.5 mm
- net Net-(ECI1-Pad4): track 0.00 -> 31.4 mm
- net Net-(ECI1-Pad5): track 0.00 -> 31.4 mm
- net Net-(ECI1-Pad3): track 0.00 -> 31.4 mm
- net Net-(ECI1-Pad2): track 0.00 -> 31.4 mm
- net Net-(D1-Pad2): track 0.00 -> 4.58 mm
- added copper zone on B.Cu, net GND
- added copper zone on F.Cu, net GND
Other:
- board outline added: 26 x 50 mm
- net class Default: trace_width 0.25 -> 0.5
- board text added: "A13"
- board text added: "A14"
- board text added: "A15"
- board text added: "ATARI 130XE BREAKOUT ECI BUS"
- board text added: "AUDIO"
- board text added: "GND"
- board text added: "NC"
- board text added: "VCC"
- board text added: "~D1XX"
- board text added: "~EXSEL"
- board text added: "~HALT"
- board text added: "~IRQ"
- board text added: "~MPD"
- board text added: "~REF"
- board text added: "~RST"
