File: ECI-Breakout.kicad_pcb (KiCad board)
At the start: 2 copper layers, 26 x 50 mm, 7 parts, among them P1 CONN_01X07, P2 CONN_01X07

Commit message: Not used
Parts:
- removed OSHW: Symbol_OSHW-Logo_SilkScreen, Symbols:Symbol_OSHW-Logo_SilkScreen
- removed kicadlogo: KiCad-Logo_5mm_SilkScreen, Symbol:KiCad-Logo_5mm_SilkScreen
- D1: value YELLOW -> LED GREEN; footprint LEDs:LED_1206 -> LED_SMD:LED_1206_3216Metric
- P1, P2: value CONN_01X07 -> Conn_01x07; footprint Pin_Headers:Pin_Header_Straight_1x07 -> Connector_PinHeader_2.54mm:PinHeader_1x07_P2.54mm_Vertical
- R1: footprint Resistors_SMD:R_1206_HandSoldering -> Resistor_SMD:R_1206_3216Metric_Pad1.30x1.75mm_HandSolder
- moved P1 0.44 mm to (139.6, 73.2)
- moved P2 0.10 mm to (139.6, 83.8)
- moved D1 0.05 mm to (135.0, 101.0)
Routing:
- net GND: track 57.3 -> 58.6 mm
- net Net-(ECI1-PadD): track 50.1 -> 51.2 mm
- net VCC: track 50.9 -> 49.9 mm
- net Net-(ECI1-PadF): track 44.7 -> 45.5 mm
- net Net-(ECI1-PadC): track 48.0 -> 48.7 mm
- net Net-(D1-Pad2): track 4.58 -> 5.09 mm

Commit message: Added NetList
Parts:
- added REF**: OSHW-Logo_5.7x6mm_SilkScreen, Symbol:OSHW-Logo_5.7x6mm_SilkScreen, B.Cu at (132.1, 95.8)
- added REF**: KiCad-Logo2_5mm_SilkScreen, Symbol:KiCad-Logo2_5mm_SilkScreen, B.Cu at (132.1, 89.2)
Connections:
- net Net-(ECI1-Pad1) renamed /~EXSEL
- net Net-(ECI1-Pad2) renamed /~RST
- net Net-(ECI1-Pad3) renamed /~D1XX
- net Net-(ECI1-Pad4) renamed /~MPD
- net Net-(ECI1-Pad5) renamed /AUDIO
- net Net-(ECI1-Pad6) renamed /~REF
- net Net-(ECI1-PadA) renamed /RSRVD
- net Net-(ECI1-PadB) renamed /~IRQ
- net Net-(ECI1-PadC) renamed /~HALT
- net Net-(ECI1-PadD) renamed /A13
- net Net-(ECI1-PadE) renamed /A14
- net Net-(ECI1-PadF) renamed /A15
Routing:
- net /A14: track 52.8 -> 54.3 mm
- net /A13: track 51.2 -> 51.9 mm
- net /RSRVD: track 46.0 -> 45.4 mm
