File: ECI-Breakout.sch (KiCad schematic (older format))
At the start: 4 parts, among them P1 CONN_02X07

Commit message: First elaborate project
Parts:
- removed P1: CONN_02X07, Connector_PinHeader_2.54mm:PinHeader_2x07_P2.54mm_Vertical, symbol CONN_02X07
- added P1, P2: CONN_01X07, Pin_Headers:Pin_Header_Straight_1x07, symbol CONN_01X07
- R1: value 330 -> 1.5K; footprint Resistors_SMD:R_1210_HandSoldering -> Resistors_SMD:R_1206_HandSoldering
Connections:
- net GND: now also P1.7 (P7)
- net VCC: now also P2.7 (P7)
- net at ECI1.1 (~EXSEL): now also P2.1 (P1)
- net at ECI1.2 (~RST): now also P2.2 (P2)
- net at ECI1.3 (~D1XX): now also P2.3 (P3)
- net at ECI1.4 (~MPD): now also P2.4 (P4)
- net at ECI1.5 (AUDIO): now also P2.5 (P5)
- net at ECI1.6 (~REF): now also P2.6 (P6)
- net at ECI1.A (RSRVD): now also P1.1 (P1)
- net at ECI1.B (~IRQ): now also P1.2 (P2)
- net at ECI1.C (~HALT): now also P1.3 (P3)
- net at ECI1.D (A13): now also P1.4 (P4)
- net at ECI1.E (A14): now also P1.5 (P5)
- net at ECI1.F (A15): now also P1.6 (P6)
Changed lines of the file:
@@
 P 7800 2850
 F 0 "R1" H 7830 2870 50  0000 L CNN
-F 1 "330" H 7830 2810 50  0000 L CNN
-F 2 "Resistors_SMD:R_1210_HandSoldering" H 7800 2850 50  0001 C CNN
+F 1 "1.5K" H 7830 2810 50  0000 L CNN
+F 2 "Resistors_SMD:R_1206_HandSoldering" H 7800 2850 50  0001 C CNN
 F 3 "" H 7800 2850 50  0000 C CNN
 	1    7800 2850
@@
 	1    0    0    -1
 $EndComp
-$Comp
-L CONN_02X07 P1
-U 1 1 5CADC0E2
-P 5600 2400
-F 0 "P1" H 5600 2800 50  0000 C CNN
-F 1 "CONN_02X07" V 5600 2400 50  0000 C CNN
-F 2 "Connector_PinHeader_2.54mm:PinHeader_2x07_P2.54mm_Vertical" H 5600 1200 50  0000 C CNN
-F 3 "" H 5600 1200 50  0000 C CNN
-	1    5600 2400
-	0    -1   -1   0
-$EndComp
 Wire Wire Line
 	4650 3450 4650 2700
@@
 Connection ~ 4500 4050
 Wire Wire Line
-	5900 2150 5900 2050
-Wire Wire Line
 	5900 2050 6500 2050
 Wire Wire Line
@@
 	6550 2000 5800 2000
 Wire Wire Line
-	5800 2000 5800 2150
-Wire Wire Line
 	6450 3650 6600 3650
 Wire Wire Line
@@
 	6600 1950 5700 1950
 Wire Wire Line
-	5700 1950 5700 2150
-Wire Wire Line
 	6450 3750 6650 3750
 Wire Wire Line
@@
 	6650 1900 5600 1900
 Wire Wire Line
-	5600 1900 5600 2150
-Wire Wire Line
 	6450 3850 6700 3850
 Wire Wire Line
@@
 	6700 1850 5500 1850
 Wire Wire Line
-	5500 1850 5500 2150
-Wire Wire Line
 	6450 3950 6750 3950
 Wire Wire Line
@@
 Wire Wire Line
 	6750 1800 5400 1800
-Wire Wire Line
-	5400 1800 5400 2150
-Wire Wire Line
-	5300 2150 5300 1750
 Wire Wire Line
 	5300 1750 6800 1750
@@
 	6800 1750 6800 4050
 Connection ~ 6600 4050
+$Comp
+L CONN_01X07 P1
+U 1 1 5CB38837
+P 5600 2300
+F 0 "P1" H 5600 2700 50  0000 C CNN
+F 1 "CONN_01X07" H 5400 1850 50  0000 C CNN
+F 2 "Pin_Headers:Pin_Header_Straight_1x07" H 5600 2300 50  0001 C CNN
+F 3 "" H 5600 2300 50  0000 C CNN
+	1    5600 2300
+	0    1    1    0
+$EndComp
+$Comp
+L CONN_01X07 P2
+U 1 1 5CB388A4
+P 5600 2450
+F 0 "P2" H 5600 2850 50  0000 C CNN
+F 1 "CONN_01X07" H 5300 2000 50  0000 C CNN
+F 2 "Pin_Headers:Pin_Header_Straight_1x07" H 5600 2450 50  0001 C CNN
+F 3 "" H 5600 2450 50  0000 C CNN
+	1    5600 2450
+	0    -1   -1   0
+$EndComp
+Wire Wire Line
+	5900 2050 5900 2100
+Wire Wire Line
+	5800 2000 5800 2100
+Wire Wire Line
+	5700 1950 5700 2100
+Wire Wire Line
+	5600 1900 5600 2100
+Wire Wire Line
+	5500 1850 5500 2100
+Wire Wire Line
+	5400 1800 5400 2100
+Wire Wire Line
+	5300 1750 5300 2100
 $EndSCHEMATC

Commit message: Update to KiCAD 5.1.19
Parts:
- removed D1: YELLOW, LEDs:LED_1206, symbol Led_Small
- removed P1, P2: CONN_01X07, Pin_Headers:Pin_Header_Straight_1x07, symbol CONN_01X07
- added D1: LED GREEN, LED_SMD:LED_1206_3216Metric, symbol Device:LED_Small_ALT
- added P1, P2: Conn_01x07, Connector_PinHeader_2.54mm:PinHeader_1x07_P2.54mm_Vertical, symbol Connector_Generic:Conn_01x07
- ECI1: symbol ECIBUS -> RetroBitLab:ECIBUS
- R1: footprint Resistors_SMD:R_1206_HandSoldering -> Resistor_SMD:R_1206_3216Metric_Pad1.30x1.75mm_HandSolder; symbol R_Small -> Device:R_Small
Connections:
- wire segments 59 -> 61

Commit message: Added NetList
Connections:
- net labels added: A13, A14, A15, AUDIO, RSRVD, ~D1XX, ~EXSEL, ~HALT, ~IRQ, ~MPD, ~REF, ~RST
- wire segments 61 -> 62
Changed lines of the file:
@@
 $EndComp
 Wire Wire Line
-	4350 4050 4500 4050
-Wire Wire Line
-	4500 4050 4500 4200
+	3375 4050 4400 4050
 $Comp
 L power:VCC #PWR04
 U 1 1 5CADC066
-P 4500 4200
-F 0 "#PWR04" H 4500 4050 50  0001 C CNN
-F 1 "VCC" H 4500 4350 50  0000 C CNN
-F 2 "" H 4500 4200 50  0001 C CNN
-F 3 "" H 4500 4200 50  0001 C CNN
-	1    4500 4200
+P 4400 4200
+F 0 "#PWR04" H 4400 4050 50  0001 C CNN
+F 1 "VCC" H 4400 4350 50  0000 C CNN
+F 2 "" H 4400 4200 50  0001 C CNN
+F 3 "" H 4400 4200 50  0001 C CNN
+	1    4400 4200
 	-1   0    0    1
 $EndComp
@@
 $EndComp
 Wire Wire Line
-	4650 3450 4650 2700
-Wire Wire Line
-	4650 2700 5300 2700
+	3675 3450 3675 2700
+Wire Wire Line
+	3675 2700 5300 2700
 Wire Wire Line
 	5300 2700 5300 2650
 Wire Wire Line
-	4650 3550 4600 3550
-Wire Wire Line
-	4600 3550 4600 2750
-Wire Wire Line
-	4600 2750 5400 2750
+	4650 3550 3625 3550
+Wire Wire Line
+	3625 3550 3625 2750
+Wire Wire Line
+	3625 2750 5400 2750
 Wire Wire Line
 	5400 2750 5400 2650
 Wire Wire Line
-	4650 3650 4550 3650
-Wire Wire Line
-	4550 3650 4550 2800
-Wire Wire Line
-	4550 2800 5500 2800
+	4650 3650 3575 3650
+Wire Wire Line
+	3575 3650 3575 2800
+Wire Wire Line
+	3575 2800 5500 2800
 Wire Wire Line
 	5500 2800 5500 2650
 Wire Wire Line
-	4650 3750 4500 3750
-Wire Wire Line
-	4500 3750 4500 2850
-Wire Wire Line
-	4500 2850 5600 2850
+	4650 3750 3525 3750
+Wire Wire Line
+	3525 3750 3525 2850
+Wire Wire Line
+	3525 2850 5600 2850
 Wire Wire Line
 	5600 2850 5600 2650
 Wire Wire Line
-	4650 3850 4450 3850
-Wire Wire Line
-	4450 3850 4450 2900
-Wire Wire Line
-	4450 2900 5700 2900
+	4650 3850 3475 3850
+Wire Wire Line
+	3475 3850 3475 2900
+Wire Wire Line
+	3475 2900 5700 2900
 Wire Wire Line
 	5700 2900 5700 2650
 Wire Wire Line
-	4650 3950 4400 3950
-Wire Wire Line
-	4400 3950 4400 2950
-Wire Wire Line
-	4400 2950 5800 2950
+	4650 3950 3425 3950
+Wire Wire Line
+	3425 3950 3425 2950
+Wire Wire Line
+	3425 2950 5800 2950
 Wire Wire Line
 	5800 2950 5800 2650
 Wire Wire Line
-	4350 4050 4350 3000
-Wire Wire Line
-	4350 3000 5900 3000
+	3375 4050 3375 3000
+Wire Wire Line
+	3375 3000 5900 3000
 Wire Wire Line
 	5900 3000 5900 2650
-Connection ~ 4500 4050
-Wire Wire Line
-	5900 2050 6500 2050
-Wire Wire Line
-	6500 2050 6500 3450
-Wire Wire Line
-	6500 3450 6450 3450
-Wire Wire Line
-	6450 3550 6550 3550
-Wire Wire Line
-	6550 3550 6550 2000
-Wire Wire Line
-	6550 2000 5800 2000
-Wire Wire Line
-	6450 3650 6600 3650
-Wire Wire Line
-	6600 3650 6600 1950
-Wire Wire Line
-	6600 1950 5700 1950
-Wire Wire Line
-	6450 3750 6650 3750
-Wire Wire Line
-	6650 3750 6650 1900
-Wire Wire Line
-	6650 1900 5600 1900
-Wire Wire Line
-	6450 3850 6700 3850
-Wire Wire Line
-	6700 3850 6700 1850
-Wire Wire Line
-	6700 1850 5500 1850
-Wire Wire Line
-	6450 3950 6750 3950
-Wire Wire Line
-	6750 3950 6750 1800
-Wire Wire Line
-	6750 1800 5400 1800
-Wire Wire Line
-	5300 1750 6800 1750
-Wire Wire Line
-	6800 1750 6800 4050
+Wire Wire Line
+	7250 2050 7250 3450
+Wire Wire Line
+	7250 3450 6450 3450
+Wire Wire Line
+	6450 3550 7300 3550
+Wire Wire Line
+	7300 3550 7300 2000
+Wire Wire Line
+	7300 2000 5800 2000
+Wire Wire Line
+	6450 3650 7350 3650
+Wire Wire Line
+	7350 3650 7350 1950
+Wire Wire Line
+	7350 1950 5700 1950
+Wire Wire Line
+	6450 3750 7400 3750
+Wire Wire Line
+	7400 3750 7400 1900
+Wire Wire Line
+	7400 1900 5600 1900
+Wire Wire Line
+	6450 3850 7450 3850
+Wire Wire Line
+	7450 3850 7450 1850
+Wire Wire Line
+	7450 1850 5500 1850
+Wire Wire Line
+	6450 3950 7500 3950
+Wire Wire Line
+	7500 3950 7500 1800
+Wire Wire Line
+	7500 1800 5400 1800
+Wire Wire Line
+	5300 1750 7550 1750
+Wire Wire Line
+	7550 1750 7550 4050
 Connection ~ 6600 4050
 Wire Wire Line
@@
 	5300 1750 5300 2100
 Wire Wire Line
-	4500 4050 4650 4050
-Wire Wire Line
-	6600 4050 6800 4050
+	6600 4050 7550 4050
 $Comp
 L Connector_Generic:Conn_01x07 P1
@@
 	0    -1   -1   0
 $EndComp
+$Comp
+L Graphic:Logo_Open_Hardware_Small #LOGO1
+U 1 1 6881E816
+P 7125 6050
+F 0 "#LOGO1" H 7125 6325 50  0001 C CNN
+F 1 "Logo_Open_Hardware_Small" H 7125 5825 50  0001 C CNN
+F 2 "" H 7125 6050 50  0001 C CNN
+F 3 "~" H 7125 6050 50  0001 C CNN
+	1    7125 6050
+	1    0    0    -1
+$EndComp
+Wire Wire Line
+	5900 2050 7250 2050
+Wire Wire Line
+	4650 3450 3675 3450
+Text Label 6650 3450 0    39   ~ 0
+RSRVD
+Text Label 6650 3550 0    39   ~ 0
+~IRQ
+Text Label 6650 3650 0    39   ~ 0
+~HALT
+Text Label 6650 3750 0    39   ~ 0
+A13
+Text Label 6650 3850 0    39   ~ 0
+A14
+Text Label 6650 3950 0    39   ~ 0
+A15
+Text Label 6650 4050 0    39   ~ 0
+GND
+Text Label 4525 3450 0    39   ~ 0
+~EXSEL
+Text Label 4525 3550 0    39   ~ 0
+~RST
+Text Label 4525 3650 0    39   ~ 0
+~D1XX
+Text Label 4525 3750 0    39   ~ 0
+~MPD
+Text Label 4525 3850 0    39   ~ 0
+AUDIO
+Text Label 4525 3950 0    39   ~ 0
+~REF
+Text Label 4525 4050 0    39   ~ 0
+VCC
+Wire Wire Line
+	4400 4200 4400 4050
+Connection ~ 4400 4050
+Wire Wire Line
+	4400 4050 4650 4050
 $EndSCHEMATC
